File: Cam-connector.kicad_sch (KiCad schematic)
At the start: 7 parts, among them J1 5051104096, J2 F304-1A7H1-11050-E100, U1 TSC2007IPW

Commit message: Small form factor
Other:
- note added: "Resistive touch screen signal to I2C."
- note removed: "Resistive to I2C"
Changed lines of the file:
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@@
 		)
 	)
-	(text "Resistive to I2C"
+	(text "Resistive touch \nscreen signal to I2C."
 		(exclude_from_sim no)
 		(at 201.93 27.305 0)
