File: Cam-connector.kicad_sch (KiCad schematic)
At the start: 7 parts, among them J1 5051104096, J2 F304-1A7H1-11050-E100, U1 TSC2007IPW

Commit message: Changes
Connections:
- net SDI is gone; now on net LCD_R0: J2.34
- net GND: no longer J2.38
- net LCD_R1: now also J2.38
- no-connect marks 9 -> 6
Other:
- note removed: "Low for parallel communication."
Changed lines of the file:
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@@
 	(generator_version "10.0")
 	(paper "A4")
-	(text "Low for parallel \ncommunication."
-		(exclude_from_sim no)
-		(at 76.2 125.73 0)
-		(effects
-			(font
-				(size 1.27 1.27)
-			)
-		)
-	)
 	(text "To control other signals, some of the pins that are used\nfor RGB data are re-mapped to control the LCD. "
 		(exclude_from_sim no)
@@
 	)
 	(no_connect
-		(at 100.33 114.935)
-	)
-	(no_connect
-		(at 29.21 59.055)
-	)
-	(no_connect
-		(at 29.21 56.515)
-	)
-	(no_connect
 		(at 29.21 61.595)
 	)
@@
 	(wire
 		(pts
-			(xy 85.725 125.095) (xy 110.49 125.095)
-		)
-		(stroke
-			(width 0)
-			(type default)
-		)
-	)
-	(wire
-		(pts
 			(xy 234.315 67.945) (xy 234.315 66.04)
 		)
@@
 	(wire
 		(pts
+			(xy 186.055 136.525) (xy 204.47 136.525)
+		)
+		(stroke
+			(width 0)
+			(type default)
+		)
+	)
+	(wire
+		(pts
 			(xy 100.33 114.935) (xy 110.49 114.935)
 		)
@@
 	(wire
 		(pts
+			(xy 186.055 133.35) (xy 204.47 133.35)
+		)
+		(stroke
+			(width 0)
+			(type default)
+		)
+	)
+	(wire
+		(pts
 			(xy 217.17 54.61) (xy 224.79 54.61)
 		)
@@
 	(wire
 		(pts
+			(xy 100.33 125.095) (xy 110.49 125.095)
+		)
+		(stroke
+			(width 0)
+			(type default)
+		)
+	)
+	(wire
+		(pts
 			(xy 224.79 54.61) (xy 224.79 57.785)
 		)
@@
 		)
 	)
+	(label "{slash}CS"
+		(at 204.47 136.525 0)
+		(effects
+			(font
+				(size 1.27 1.27)
+			)
+			(justify left bottom)
+		)
+	)
 	(label "LCD_RST"
 		(at 186.055 117.475 0)
@@
 		)
 	)
+	(label "LCD_R0"
+		(at 186.055 133.35 0)
+		(effects
+			(font
+				(size 1.27 1.27)
+			)
+			(justify left bottom)
+		)
+	)
 	(label "DB2"
 		(at 100.33 104.775 0)
@@
 		)
 	)
+	(label "LCD_R1"
+		(at 186.055 136.525 0)
+		(effects
+			(font
+				(size 1.27 1.27)
+			)
+			(justify left bottom)
+		)
+	)
 	(label "IOVCC"
 		(at 100.33 132.715 0)
@@
 		)
 	)
+	(label "SDI"
+		(at 204.47 133.35 0)
+		(effects
+			(font
+				(size 1.27 1.27)
+			)
+			(justify left bottom)
+		)
+	)
 	(label "DE"
 		(at 205.105 120.65 0)
@@
 					(unit 1)
 				)
-			)
-		)
-	)
-	(symbol
-		(lib_id "power:GND")
-		(at 85.725 125.095 0)
-		(unit 1)
-		(body_style 1)
-		(exclude_from_sim no)
-		(in_bom yes)
-		(on_board yes)
-		(in_pos_files yes)
-		(dnp no)
-		(fields_autoplaced yes)
-		(property "Reference" "#PWR018"
-			(at 85.725 131.445 0)
-			(hide yes)
-			(show_name no)
-			(do_not_autoplace no)
-			(effects
-				(font
-					(size 1.27 1.27)
-				)
-			)
-		)
-		(property "Value" "GND"
-			(at 85.725 129.54 0)
-			(show_name no)
-			(do_not_autoplace no)
-			(effects
-				(font
-					(size 1.27 1.27)
-				)
-			)
-		)
-		(property "Footprint" ""
-			(at 85.725 125.095 0)
-			(hide yes)
-			(show_name no)
-			(do_not_autoplace no)
-			(effects
-				(font
-					(size 1.27 1.27)
-				)
-			)
-		)
-		(property "Datasheet" ""
-			(at 85.725 125.095 0)
-			(hide yes)
-			(show_name no)
-			(do_not_autoplace no)
-			(effects
-				(font
-					(size 1.27 1.27)
-				)
-			)
-		)
-		(property "Description" "Power symbol creates a global label with name \"GND\" , ground"
-			(at 85.725 125.095 0)
-			(hide yes)
-			(show_name no)
-			(do_not_autoplace no)
-			(effects
-				(font
-					(size 1.27 1.27)
-				)
-			)
-		)
-		(pin "1"
-		)
-		(instances
-			(project "Cam-connector"
-				(path "/3f2f492d-9b77-43e2-b336-8c59a538cbe4"
-					(reference "#PWR018")
-					(unit 1)
-				)
