File: Cam-connector.kicad_sch (KiCad schematic)
At the start: 8 parts, among them J1 5051104096, J2 F304-1A7H1-11050-E100, J3 Conn_01x02_Pin, U1 TSC2007IPW

Commit message: V1.1
Parts:
- J1: footprint footprints:CON_5051104096_MOL -> Connector_FFC-FPC:Hirose_FH12-40S-0.5SH_1x40-1MP_P0.50mm_Horizontal
- J2: footprint footprints:AMPHENOL_F304-1A7H1-11050-E100 -> Connector_FFC-FPC:Hirose_FH12-50S-0.5SH_1x50-1MP_P0.50mm_Horizontal
Connections:
- no-connect marks 5 -> 12
Changed lines of the file:
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@@
 	)
 	(no_connect
+		(at 29.21 130.175)
+	)
+	(no_connect
 		(at 29.21 61.595)
 	)
 	(no_connect
+		(at 29.21 127.635)
+	)
+	(no_connect
+		(at 29.21 76.835)
+	)
+	(no_connect
+		(at 29.21 99.695)
+	)
+	(no_connect
+		(at 29.21 79.375)
+	)
+	(no_connect
 		(at 100.33 127.635)
 	)
 	(no_connect
+		(at 29.21 97.155)
+	)
+	(no_connect
 		(at 100.33 117.475)
 	)
@@
 		(at 196.215 122.555)
 	)
+	(no_connect
+		(at 29.21 102.235)
+	)
 	(wire
 		(pts
@@
 			)
 		)
-		(property "Footprint" "footprints:CON_5051104096_MOL"
+		(property "Footprint" "Connector_FFC-FPC:Hirose_FH12-40S-0.5SH_1x40-1MP_P0.50mm_Horizontal"
 			(at 41.275 43.815 0)
 			(hide yes)
@@
 			)
 		)
-		(property "Footprint" "footprints:AMPHENOL_F304-1A7H1-11050-E100"
+		(property "Footprint" "Connector_FFC-FPC:Hirose_FH12-50S-0.5SH_1x50-1MP_P0.50mm_Horizontal"
 			(at 120.65 94.615 0)
 			(hide yes)
