File: Cam-connector.kicad_sch (KiCad schematic)
At the start: 7 parts, among them J1 5051104096, J2 F304-1A7H1-11050-E100, U1 TSC2007IPW

Commit message: V1.1
Parts:
- removed JP1, JP2: SolderJumper_2_Open, Jumper:SolderJumper-2_P1.3mm_Open_TrianglePad1.0x1.5mm, symbol Jumper:SolderJumper_2_Open
- added J3: Conn_01x02_Pin, Connector_PinHeader_2.54mm:PinHeader_1x02_P2.54mm_Vertical, symbol Connector:Conn_01x02_Pin
- added R3, R4: 10k, Resistor_SMD:R_0603_1608Metric, symbol Device:R
- J1: footprint Parts:CON_5051104096_MOL -> Connector_FFC-FPC:Hirose_FH12-40S-0.5SH_1x40-1MP_P0.50mm_Horizontal
- J2: footprint Parts:AMPHENOL_F304-1A7H1-11050-E100 -> Connector_FFC-FPC:Hirose_FH12-50S-0.5SH_1x50-1MP_P0.50mm_Horizontal
- R1, R2: footprint Resistor_SMD:R_0402_1005Metric -> Resistor_SMD:R_0603_1608Metric
Connections:
- net LDC_SDA is gone; now on net LCD_SDA: J1.39
- net DB1: now also J1.25; no longer J1.26
- net DB10: now also J1.20; no longer J1.21
- net DB11: now also J1.21; no longer J1.9
- net DB13: now also J1.9; no longer J1.11
- net DB14: now also J1.10; no longer J1.12
- net DB15: now also J1.11; no longer J1.13
- net DB2: now also J1.26; no longer J1.27
- net DB3: now also J1.27; no longer J1.28
- net DB4: now also J1.28; no longer J1.29
- net DB5: now also J1.29; no longer J1.16
- net DB6: now also J1.16; no longer J1.17
- net DB7: now also J1.17; no longer J1.18
- net DB8: now also J1.18; no longer J1.19
- net DB9: now also J1.19; no longer J1.20
- net GND: now also J2.20, J2.32, J2.6; no longer J2.15, J2.16, J2.38, J2.7, J2.8
- net LCD_B0: no longer J2.35
- net LCD_B1: no longer J2.36
- net LCD_B2: no longer J2.37
- net LCD_R0: now also J2.38
- net LCD_R1: now also J2.36
- net LCD_SCL: now also R4.2
- net LCD_SDA: now also R3.2
- net SYS_3V3: now also J2.7, J2.8, R3.1, R4.1; no longer J2.6
- removed net DB0: J1.25, J2.32
- removed net DB12: J1.10, J2.20
- net LCD_R57 renamed UHH IDK
- net SDI renamed MOSI
- net MOSI: now also J3.1 (Pin_1)
- new net DB16: J1.12, J2.16
- new net DB17: J1.13, J2.15
- new net RS_SCL: J2.37, J3.2 (Pin_2)
- new net /RD: J2.35
- no-connect marks 9 -> 12
Other:
- note added: "Corresponds to 16-bit parallel interface. "0110""
- note added: "SPI Data"
- note added: "Sync Data"
- note removed: "Control data"
- note removed: "Corresponds to 16-bit parallel interface. "0001""
- note removed: "Low for parallel communication."
- note removed: "To control other signals, some of the pins that are used for RGB data are re-mapped to control the LCD."
- moved on the sheet: U1
