File: Cam-connector.kicad_pcb (KiCad board)
At the start: 2 copper layers, 34.5 x 26.4 mm, 7 parts, among them J1 5051104096, J2 F304-1A7H1-11050-E100, U1 TSC2007IPW

Commit message: V1.1
Parts:
- removed JP1, JP2: SolderJumper_2_Open, Jumper:SolderJumper-2_P1.3mm_Open_TrianglePad1.0x1.5mm
- added J3: Conn_01x02_Pin, Connector_PinHeader_2.54mm:PinHeader_1x02_P2.54mm_Vertical, F.Cu at (136.3, 69.3)
- added R3: 10k, Resistor_SMD:R_0603_1608Metric, B.Cu at (130.2, 60.8)
- added R4: 10k, Resistor_SMD:R_0603_1608Metric, B.Cu at (130.2, 62.4)
- J1: footprint Parts:CON_5051104096_MOL -> Connector_FFC-FPC:Hirose_FH12-40S-0.5SH_1x40-1MP_P0.50mm_Horizontal
- J2: footprint Parts:AMPHENOL_F304-1A7H1-11050-E100 -> Connector_FFC-FPC:Hirose_FH12-50S-0.5SH_1x50-1MP_P0.50mm_Horizontal
- R1, R2: footprint Resistor_SMD:R_0402_1005Metric -> Resistor_SMD:R_0603_1608Metric; moved to B.Cu
- U1: moved to B.Cu
- moved U1 50.0 mm to (124.7, 63.3), turned to 0 degrees
- moved R1 39.6 mm to (130.2, 64.0)
- moved R2 37.1 mm to (130.2, 65.7)
- moved J1 35.8 mm to (125.0, 74.3), turned to 0 degrees
- moved J2 35.0 mm to (125.0, 64.5), turned to 180 degrees
Connections:
- net /LCD_R57 renamed /UHH IDK
- J1 pad 10: /DB12 -> /DB14
- J1 pad 11: /DB13 -> /DB15
- J1 pad 12: /DB14 -> /DB16
- J1 pad 13: /DB15 -> /DB17
- J1 pad 16: /DB5 -> /DB6
- J1 pad 17: /DB6 -> /DB7
- J1 pad 18: /DB7 -> /DB8
- J1 pad 19: /DB8 -> /DB9
- J1 pad 20: /DB9 -> /DB10
- J1 pad 21: /DB10 -> /DB11
- J1 pad 25: /DB0 -> /DB1
- J1 pad 26: /DB1 -> /DB2
- J1 pad 27: /DB2 -> /DB3
- J1 pad 28: /DB3 -> /DB4
- J1 pad 29: /DB4 -> /DB5
- J1 pad 39: /LDC_SDA -> /LCD_SDA
- J1 pad 9: /DB11 -> /DB13
- J2 pad 15: GND -> /DB17
- J2 pad 16: GND -> /DB16
- J2 pad 20: /DB12 -> GND
- J2 pad 32: /DB0 -> GND
- J2 pad 34: /SDI -> /MOSI
- J2 pad 35: /LCD_B0 -> //RD
- J2 pad 36: /LCD_B1 -> /LCD_R1
- J2 pad 37: /LCD_B2 -> /RS_SCL
- J2 pad 38: GND -> /LCD_R0
- J2 pad 6: SYS_3V3 -> GND
- J2 pad 7: GND -> SYS_3V3
- J2 pad 8: GND -> SYS_3V3
Routing:
- net /RS_SCL: track 0.00 -> 25.4 mm
- net /LCD_B2: track 24.7 -> 0.00 mm, vias 2 -> 0
- net /LCD_B1: track 24.6 -> 0.00 mm, vias 2 -> 0
- net /DB12: track 24.4 -> 0.00 mm, vias 2 -> 0
- net /DB0: track 24.3 -> 0.00 mm, vias 2 -> 0
- net /DB16: track 0.00 -> 24.1 mm, vias 0 -> 2
- net /MOSI: track 0.00 -> 24.0 mm
- net /LCD_B0: track 23.7 -> 0.00 mm, vias 2 -> 0
- net /DB17: track 0.00 -> 23.0 mm, vias 0 -> 2
- net SYS_3V3: track 26.1 -> 48.6 mm, vias 8 -> 4
- net /LCD_SDA: track 0.00 -> 21.0 mm, vias 0 -> 1
- net /DB11: track 24.3 -> 7.05 mm, vias 2 -> 0
- net /LCD_SCL: track 31.6 -> 15.8 mm, vias 0 -> 1
- net /DB4: track 24.8 -> 10.7 mm
- net /DB10: track 21.1 -> 7.05 mm
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- removed copper zone on F.Cu, net SYS_3V3
Other:
- board size 34.5 x 26.4 mm -> 32.3 x 19.8 mm
- board text added: "MOSI SCLK"
- board text added: "Stanley Barnes, EPIC Lab at UTK Screen Connector V1.1 Wio Lite Ai 40-pin to 3.2{dblquote} Adafruit TFT 50-pin"
- board text added: "Touchscreen"
- board text added: "Wio Lite Ai"
