File: Cam-connector.kicad_pcb (KiCad board)
At the start: 2 copper layers, 34.8 x 38.2 mm, 7 parts, among them J1 5051104096, J2 F304-1A7H1-11050-E100, U1 TSC2007IPW

Commit message: V1.1
Parts:
- removed JP1, JP2: SolderJumper_2_Open, Jumper:SolderJumper-2_P1.3mm_Open_TrianglePad1.0x1.5mm
- added J3: Conn_01x02_Pin, Connector_PinHeader_2.54mm:PinHeader_1x02_P2.54mm_Vertical, F.Cu at (169.4, 65.7)
- added R3: 10k, Resistor_SMD:R_0603_1608Metric, F.Cu at (147.4, 80.6)
- added R4: 10k, Resistor_SMD:R_0603_1608Metric, F.Cu at (145.8, 80.6)
- J1: footprint Parts:CON_5051104096_MOL -> Connector_FFC-FPC:Hirose_FH12-40S-0.5SH_1x40-1MP_P0.50mm_Horizontal
- J2: footprint Parts:AMPHENOL_F304-1A7H1-11050-E100 -> Connector_FFC-FPC:Hirose_FH12-50S-0.5SH_1x50-1MP_P0.50mm_Horizontal
- R1, R2: footprint Resistor_SMD:R_0402_1005Metric -> Resistor_SMD:R_0603_1608Metric
- moved R2 30.0 mm to (142.2, 79.5), turned to 180 degrees
- moved R1 29.4 mm to (142.3, 81.1), turned to 180 degrees
- moved U1 25.3 mm to (145.2, 72.6), turned to 0 degrees
- moved J1 1.00 mm to (157.2, 87.9), turned to 0 degrees
- moved J2 0.36 mm to (157.0, 60.0), turned to 180 degrees
Connections:
- net /LCD_R57 renamed /UHH IDK
- J1 pad 10: /DB12 -> /DB14
- J1 pad 11: /DB13 -> /DB15
- J1 pad 12: /DB14 -> /DB16
- J1 pad 13: /DB15 -> /DB17
- J1 pad 16: /DB5 -> /DB6
- J1 pad 17: /DB6 -> /DB7
- J1 pad 18: /DB7 -> /DB8
- J1 pad 19: /DB8 -> /DB9
- J1 pad 20: /DB9 -> /DB10
- J1 pad 21: /DB10 -> /DB11
- J1 pad 25: /DB0 -> /DB1
- J1 pad 26: /DB1 -> /DB2
- J1 pad 27: /DB2 -> /DB3
- J1 pad 28: /DB3 -> /DB4
- J1 pad 29: /DB4 -> /DB5
- J1 pad 39: /LDC_SDA -> /LCD_SDA
- J1 pad 9: /DB11 -> /DB13
- J2 pad 15: GND -> /DB17
- J2 pad 16: GND -> /DB16
- J2 pad 20: /DB12 -> GND
- J2 pad 32: /DB0 -> GND
- J2 pad 34: /SDI -> /MOSI
- J2 pad 35: /LCD_B0 -> //RD
- J2 pad 36: /LCD_B1 -> /LCD_R1
- J2 pad 37: /LCD_B2 -> /RS_SCL
- J2 pad 38: GND -> /LCD_R0
- J2 pad 6: SYS_3V3 -> GND
- J2 pad 7: GND -> SYS_3V3
- J2 pad 8: GND -> SYS_3V3
Routing:
- net GND: track 100.9 -> 36.4 mm, vias 5 -> 6
- net /DB12: track 49.9 -> 0.00 mm, vias 2 -> 0
- net /LCD_SDA: track 0.00 -> 41.9 mm, vias 0 -> 2
- net /LCD_B1: track 39.2 -> 0.00 mm, vias 2 -> 0
- net /DB17: track 0.00 -> 38.8 mm, vias 0 -> 2
- net /LCD_B0: track 38.7 -> 0.00 mm, vias 2 -> 0
- net /DB16: track 0.00 -> 38.4 mm, vias 0 -> 2
- net /LCD_B2: track 37.3 -> 0.00 mm, vias 2 -> 0
- net /DB0: track 37.2 -> 0.00 mm, vias 2 -> 0
- net /RS_SCL: track 0.00 -> 30.2 mm
- net /DB11: track 50.6 -> 25.1 mm, vias 2 -> 0
- net /LCD_R0: track 0.00 -> 25.5 mm
- net /LCD_R1: track 0.00 -> 25.4 mm
- net /MOSI: track 0.00 -> 25.0 mm
- net /LCD_RST: track 37.3 -> 24.5 mm
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- added copper zone on B.Cu, net GND
- added copper zone on F.Cu, net GND
